Commit message: nicer quadrotor meshes

File: ros2_ws/src/trajectory_visualization/description/quadrotor_baseline.urdf (robot description, URDF)
Before this commit: robot Quadrotor, 1 links, 0 joints
Links:
- link baseline/body: mass 0.556 -> None; geometry visual mesh filename=file:///home/jake/Projects/EQTrackingControl/ros2_ws/src/tr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; visual mesh filename=file:///home/jake/Projects/EQTrackingControl/ros2_ws/src/tr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

File: ros2_ws/src/trajectory_visualization/description/quadrotor_symmetry.urdf (robot description, URDF)
Before this commit: robot Quadrotor, 1 links, 0 joints
Links:
- link symmetry/body: mass 0.556 -> None; geometry visual mesh filename=file:///home/jake/Projects/EQTrackingControl/ros2_ws/src/tr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; visual mesh filename=file:///home/jake/Projects/EQTrackingControl/ros2_ws/src/tr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
