Commit message: updated paths to absolute location on jakes machine

File: ros2_ws/src/trajectory_visualization/description/astrobee_baseline.urdf (robot description, URDF)
Before this commit: robot astrobee, 1 links, 0 joints
Links:
- link /baseline/body: geometry collision box size=0.290513 0.151942 0.281129; collision box size=0.319199 0.083962 0.319588

File: ros2_ws/src/trajectory_visualization/description/astrobee_symmetry.urdf (robot description, URDF)
Before this commit: robot astrobee, 1 links, 0 joints
Links:
- link /symmetry/body: geometry collision box size=0.290513 0.151942 0.281129; collision box size=0.319199 0.083962 0.319588

Commit message: resolve merge and add docs

File: ros2_ws/src/trajectory_visualization/description/astrobee_baseline.urdf (robot description, URDF)
Before this commit: robot astrobee, 1 links, 0 joints
Links:
- link /baseline/body: geometry collision box size=0.290513 0.151942 0.281129; collision box size=0.319199 0.083962 0.319588

File: ros2_ws/src/trajectory_visualization/description/astrobee_reference.urdf (robot description, URDF)
Before this commit: robot astrobee, 1 links, 0 joints
Links:
- link /reference/body: geometry collision box size=0.290513 0.151942 0.281129; collision box size=0.319199 0.083962 0.319588

File: ros2_ws/src/trajectory_visualization/description/astrobee_symmetry.urdf (robot description, URDF)
Before this commit: robot astrobee, 1 links, 0 joints
Links:
- link /symmetry/body: geometry collision box size=0.290513 0.151942 0.281129; collision box size=0.319199 0.083962 0.319588

Commit message: Pre-ICRA update

File: ros2_ws/src/trajectory_visualization/description/astrobee_baseline.urdf (robot description, URDF)
Before this commit: robot astrobee, 1 links, 0 joints
Links:
- link /baseline/body: geometry collision box size=0.290513 0.151942 0.281129; collision box size=0.319199 0.083962 0.319588

File: ros2_ws/src/trajectory_visualization/description/astrobee_reference.urdf (robot description, URDF)
Before this commit: robot astrobee, 1 links, 0 joints
Links:
- link /reference/body: geometry collision box size=0.290513 0.151942 0.281129; collision box size=0.319199 0.083962 0.319588

File: ros2_ws/src/trajectory_visualization/description/astrobee_symmetry.urdf (robot description, URDF)
Before this commit: robot astrobee, 1 links, 0 joints
Links:
- link /symmetry/body: geometry collision box size=0.290513 0.151942 0.281129; collision box size=0.319199 0.083962 0.319588

File: ros2_ws/src/trajectory_visualization/description/quadrotor_baseline.urdf (robot description, URDF)
Before this commit: robot Quadrotor, 1 links, 0 joints
Links:
- link baseline/body: geometry visual mesh filename=file:///home/pratikk/EQTrackingControl/ros2_ws/src/trajecto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; visual mesh filename=file:///home/pratikk/EQTrackingControl/ros2_ws/src/trajecto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

File: ros2_ws/src/trajectory_visualization/description/quadrotor_reference.urdf (robot description, URDF)
Before this commit: robot Quadrotor, 1 links, 0 joints
Links:
- link reference/body: geometry visual mesh filename=file:///home/pratikk/EQTrackingControl/ros2_ws/src/trajecto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; visual mesh filename=file:///home/pratikk/EQTrackingControl/ros2_ws/src/trajecto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

File: ros2_ws/src/trajectory_visualization/description/quadrotor_symmetry.urdf (robot description, URDF)
Before this commit: robot Quadrotor, 1 links, 0 joints
Links:
- link symmetry/body: geometry visual mesh filename=file:///home/pratikk/EQTrackingControl/ros2_ws/src/trajecto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; visual mesh filename=file:///home/pratikk/EQTrackingControl/ros2_ws/src/trajecto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
